Commit message: 模型添加base_footprint，避免加载模型warn

File: src/robot_description/urdf/simple_robot.urdf.xacro (robot description, xacro)
@@ -3,4 +3,5 @@
     name="simple_robot"
     xmlns:xacro="http://www.ros.org/wiki/xacro">
+    <link name="base_footprint"/>
     <link name="base_link">
         <visual>
@@ -28,3 +29,9 @@
         </inertial>
     </link>
+    <joint name="base_footprint_to_base_link" type="fixed">
+        <parent link="base_footprint"/>
+        <child link="base_link"/>
+        <origin xyz="0 0 0"
+                rpy="0 0 0"/>
+    </joint>
 </robot>

Commit message: 添加相机

File: src/robot_description/urdf/simple_robot.urdf.xacro (robot description, xacro)
@@ -35,3 +35,18 @@
                 rpy="0 0 0"/>
     </joint>
+    <link name="camera_link">
+        <visual>
+            <origin xyz="0 0 0"
+                    rpy="0 0 0"/>
+            <geometry>
+                <box size="0.05 0.05 0.05"/>
+            </geometry>
+        </visual>
+    </link>
+    <joint name="base_link_to_camera_link" type="fixed">
+        <parent link="base_link"/>
+        <child link="camera_link"/>
+        <origin xyz="0 0 0.3"
+                rpy="0 0 0"/>
+    </joint>
 </robot>

Commit message: 添加左轮

File: src/robot_description/urdf/simple_robot.urdf.xacro (robot description, xacro)
@@ -50,3 +50,23 @@
                 rpy="0 0 0"/>
     </joint>
+    <link name="left_wheel_link">
+        <visual>
+            <origin xyz="0 0.15 -0.05"
+                    rpy="1.5708 0 0"/>
+            <geometry>
+                <cylinder radius="0.05" length="0.03"/>
+            </geometry>
+            <material name="black">
+                <color rgba="0.1 0.1 0.1 1.0"/>
+            </material>
+        </visual>
+    </link>
+    <joint name="base_link_to_left_wheel_link"
+            type="continuous">
+        <parent link="base_link"/>
+        <child link="left_wheel_link"/>
+        <origin xyz="0 0 0"
+                rpy="0 0 0"/>
+        <axis xyz="0 1 0"/>
+    </joint>
 </robot>

Commit message: 添加右轮

File: src/robot_description/urdf/simple_robot.urdf.xacro (robot description, xacro)
@@ -70,3 +70,23 @@
         <axis xyz="0 1 0"/>
     </joint>
+    <link name="right_wheel_link">
+        <visual>
+            <origin xyz="0 -0.15 -0.05"
+                    rpy="1.5708 0 0"/>
+            <geometry>
+                <cylinder radius="0.05" length="0.03"/>
+            </geometry>
+            <material name="black">
+                <color rgba="0.1 0.1 0.1 1.0"/>
+            </material>
+        </visual>
+    </link>
+    <joint name="base_link_to_right_wheel_link"
+            type="continuous">
+        <parent link="base_link"/>
+        <child link="right_wheel_link"/>
+        <origin xyz="0 0 0"
+                rpy="0 0 0"/>
+        <axis xyz="0 1 0"/>
+    </joint>
 </robot>

Commit message: 修复轮子旋转轴bug

File: src/robot_description/urdf/simple_robot.urdf.xacro (robot description, xacro)
@@ -52,6 +52,6 @@
     <link name="left_wheel_link">
         <visual>
-            <origin xyz="0 0.15 -0.05"
-                    rpy="1.5708 0 0"/>
+            <origin xyz="0 0 0"
+                    rpy="1.508 0 0"/>
             <geometry>
                 <cylinder radius="0.05" length="0.03"/>
@@ -66,5 +66,5 @@
         <parent link="base_link"/>
         <child link="left_wheel_link"/>
-        <origin xyz="0 0 0"
+        <origin xyz="0 0.15 -0.05"
                 rpy="0 0 0"/>
         <axis xyz="0 1 0"/>
@@ -72,5 +72,5 @@
     <link name="right_wheel_link">
         <visual>
-            <origin xyz="0 -0.15 -0.05"
+            <origin xyz="0 0 0"
                     rpy="1.5708 0 0"/>
             <geometry>
@@ -86,5 +86,5 @@
         <parent link="base_link"/>
         <child link="right_wheel_link"/>
-        <origin xyz="0 0 0"
+        <origin xyz="0 -0.15 -0.05"
                 rpy="0 0 0"/>
         <axis xyz="0 1 0"/>
