Commit message: 加入ros2_control

File: src/robot_description/urdf/simple_robot.urdf.xacro (robot description, xacro)
@@ -90,3 +90,26 @@
         <axis xyz="0 1 0"/>
     </joint>
+    <ros2_control
+        name="GazeboSystem"
+        type="System">
+        <hardware>
+            <plugin>gz_ros2_control/GazeboSimSystem</plugin>
+        </hardware>
+        <joint name="base_link_to_left_wheel_link">
+            <command_interface name="velocity"/>
+            <state_interface name="position"/>
+            <state_interface name="velocity"/>
+        </joint>
+        <joint name="base_link_to_right_wheel_link">
+            <command_interface name="velocity"/>
+            <state_interface name="position"/>
+            <state_interface name="velocity"/>
+        </joint>
+    </ros2_control>
+    <gazebo>
+        <plugin filename="gz_ros2_control-system"
+                name="gz_ros2_control::GazeboSimROS2ControlPlugin">
+            <parameters>$(find robot_description)/config/controllers.yaml</parameters>
+        </plugin>
+    </gazebo>
 </robot>

Commit message: 修改模型，使其全部在地面上

File: src/robot_description/urdf/simple_robot.urdf.xacro (robot description, xacro)
@@ -3,8 +3,11 @@
     name="simple_robot"
     xmlns:xacro="http://www.ros.org/wiki/xacro">
+    <xacro:property
+        name="controllers_file"
+        value="$(find robot_description)/config/controllers.yaml"/>
     <link name="base_footprint"/>
     <link name="base_link">
         <visual>
-            <origin xyz="0 0 0.1"
+            <origin xyz="0 0 0"
                     rpy="0 0 0"/>
             <geometry>
@@ -13,5 +16,5 @@
         </visual>
         <collision>
-            <origin xyz="0 0 0.1"
+            <origin xyz="0 0 0"
                     rpy="0 0 0"/>
             <geometry>
@@ -20,5 +23,5 @@
         </collision>
         <inertial>
-            <origin xyz="0 0 0.1"
+            <origin xyz="0 0 0"
                     rpy="0 0 0"/>
             <mass value="1.0"/>
@@ -32,5 +35,5 @@
         <parent link="base_footprint"/>
         <child link="base_link"/>
-        <origin xyz="0 0 0"
+        <origin xyz="0 0 0.2"
                 rpy="0 0 0"/>
     </joint>
@@ -53,5 +56,5 @@
         <visual>
             <origin xyz="0 0 0"
-                    rpy="1.508 0 0"/>
+                    rpy="1.5708 0 0"/>
             <geometry>
                 <cylinder radius="0.05" length="0.03"/>
@@ -61,4 +64,20 @@
             </material>
         </visual>
+        <collision>
+            <origin xyz="0 0 0"
+                    rpy="1.5708 0 0"/>
+            <geometry>
+                <cylinder radius="0.05" length="0.03"/>
+            </geometry>
+        </collision>
+        <inertial>
+            <origin xyz="0 0 0"
+                    rpy="0 0 0"/>
+            <mass value="0.1"/>
+            <inertia
+                ixx="0.000083" ixy="0.0" ixz="0.0"
+                iyy="0.000083" iyz="0.0"
+                izz="0.000125"/>
+        </inertial>
     </link>
     <joint name="base_link_to_left_wheel_link"
@@ -66,5 +85,5 @@
         <parent link="base_link"/>
         <child link="left_wheel_link"/>
-        <origin xyz="0 0.15 -0.05"
+        <origin xyz="0 0.15 -0.15"
                 rpy="0 0 0"/>
         <axis xyz="0 1 0"/>
@@ -81,4 +100,20 @@
             </material>
         </visual>
+        <collision>
+            <origin xyz="0 0 0"
+                    rpy="1.5708 0 0"/>
+            <geometry>
+                <cylinder radius="0.05" length="0.03"/>
+            </geometry>
+        </collision>
+        <inertial>
+            <origin xyz="0 0 0"
+                    rpy="0 0 0"/>
+            <mass value="0.1"/>
+            <inertia
+                ixx="0.000083" ixy="0.0" ixz="0.0"
+                iyy="0.000083" iyz="0.0"
+                izz="0.000125"/>
+        </inertial>
     </link>
     <joint name="base_link_to_right_wheel_link"
@@ -86,11 +121,38 @@
         <parent link="base_link"/>
         <child link="right_wheel_link"/>
-        <origin xyz="0 -0.15 -0.05"
+        <origin xyz="0 -0.15 -0.15"
                 rpy="0 0 0"/>
         <axis xyz="0 1 0"/>
     </joint>
+    <link name="caster_link">
+        <visual>
+            <origin xyz="0 0 0" rpy="0 0 0"/>
+            <geometry>
+                <sphere radius="0.05"/>
+            </geometry>
+        </visual>
+        <collision>
+            <origin xyz="0 0 0" rpy="0 0 0"/>
+            <geometry>
+                <sphere radius="0.05"/>
+            </geometry>
+        </collision>
+        <inertial>
+            <origin xyz="0 0 0" rpy="0 0 0"/>
+            <mass value="0.05"/>
+            <inertia
+                ixx="0.0000125" ixy="0.0" ixz="0.0"
+                iyy="0.0000125" iyz="0.0"
+                izz="0.0000125"/>
+        </inertial>
+    </link>
+    <joint name="base_link_to_caster_link" type="fixed">
+        <parent link="base_link"/>
+        <child link="caster_link"/>
+        <origin xyz="-0.15 0 -0.15" rpy="0 0 0"/>
+    </joint>
     <ros2_control
         name="GazeboSystem"
-        type="System">
+        type="system">
         <hardware>
             <plugin>gz_ros2_control/GazeboSimSystem</plugin>
@@ -110,5 +172,5 @@
         <plugin filename="gz_ros2_control-system"
                 name="gz_ros2_control::GazeboSimROS2ControlPlugin">
-            <parameters>$(find robot_description)/config/controllers.yaml</parameters>
+            <parameters>/home/cheng/ros_ws/controllers.yaml</parameters>
         </plugin>
     </gazebo>

Commit message: 添加README文件

File: src/robot_description/urdf/simple_robot.urdf.xacro (robot description, xacro)
@@ -38,19 +38,5 @@
                 rpy="0 0 0"/>
     </joint>
-    <link name="camera_link">
-        <visual>
-            <origin xyz="0 0 0"
-                    rpy="0 0 0"/>
-            <geometry>
-                <box size="0.05 0.05 0.05"/>
-            </geometry>
-        </visual>
-    </link>
-    <joint name="base_link_to_camera_link" type="fixed">
-        <parent link="base_link"/>
-        <child link="camera_link"/>
-        <origin xyz="0 0 0.3"
-                rpy="0 0 0"/>
-    </joint>
+    <xacro:include filename="$(find robot_description)/urdf/camera.xacro"/>
     <link name="left_wheel_link">
         <visual>
