Commit message: 添加Camera Sensor

File: src/robot_description/urdf/camera.xacro (robot description, xacro)
@@ -19,5 +19,5 @@
             <origin xyz="0 0 0" rpy="0 0 0"/>
             <mass value="0.05"/>
-            <inerta
+            <inertia
                 ixx="0.00003"
                 ixy="0.0"

File: src/robot_description/urdf/simple_robot.urdf.xacro (robot description, xacro)
@@ -39,4 +39,5 @@
     </joint>
     <xacro:include filename="$(find robot_description)/urdf/camera.xacro"/>
+    <xacro:include filename="$(find robot_description)/urdf/gazebo_sensors.xacro"/>
     <link name="left_wheel_link">
         <visual>
